File: PCB_Design/Suspension_telemetry/STM32F446RET6_Base.kicad_sch (KiCad schematic)
At the start: 28 parts, among them J2 Conn_01x03_Pin, J5 HBHR-B2-10-VG-SMT, U1 STM32F446RET6, Y1 Crystal_GND24_Small, Y2 ABS07-32.768KHZ-9-T

Commit message: PCB: Finished
Other:
- moved on the sheet: C22
Changed lines of the file:
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@@
     (stroke (width 0) (type default))
   )
-  (wire (pts (xy 80.01 158.75) (xy 80.01 172.72))
+  (wire (pts (xy 77.47 162.56) (xy 77.47 172.72))
     (stroke (width 0) (type default))
   )
@@
     (stroke (width 0) (type default))
   )
-  (wire (pts (xy 80.01 172.72) (xy 105.41 172.72))
+  (wire (pts (xy 77.47 172.72) (xy 105.41 172.72))
     (stroke (width 0) (type default))
   )
@@
     (stroke (width 0) (type default))
   )
-  (wire (pts (xy 80.01 149.86) (xy 87.63 149.86))
+  (wire (pts (xy 77.47 149.86) (xy 87.63 149.86))
     (stroke (width 0) (type default))
   )
@@
     (stroke (width 0) (type default))
   )
-  (wire (pts (xy 80.01 153.67) (xy 80.01 149.86))
+  (wire (pts (xy 77.47 157.48) (xy 77.47 149.86))
     (stroke (width 0) (type default))
   )
@@
     )
   )
-  (symbol (lib_id "Device:C_Small") (at 80.01 156.21 0) (unit 1)
-    (in_bom yes) (on_board yes) (dnp no) (fields_autoplaced)
-    (property "Reference" "C22" (at 83.312 154.9463 0)
-      (effects (font (size 1.27 1.27)) (justify left))
-    )
-    (property "Value" "4,7uF" (at 83.312 157.4863 0)
-      (effects (font (size 1.27 1.27)) (justify left))
-    )
-    (property "Footprint" "Capacitor_SMD:C_0603_1608Metric_Pad1.08x0.95mm_HandSolder" (at 80.01 156.21 0)
-      (effects (font (size 1.27 1.27)) hide)
-    )
-    (property "Datasheet" "~" (at 80.01 156.21 0)
-      (effects (font (size 1.27 1.27)) hide)
-    )
+  (symbol (lib_id "Device:C_Small") (at 77.47 160.02 0) (unit 1)
+    (in_bom yes) (on_board yes) (dnp no) (fields_autoplaced)
+    (property "Reference" "C22" (at 80.772 158.7563 0)
+      (effects (font (size 1.27 1.27)) (justify left))
+    )
+    (property "Value" "4,7uF" (at 80.772 161.2963 0)
+      (effects (font (size 1.27 1.27)) (justify left))
+    )
+    (property "Footprint" "Capacitor_SMD:C_0603_1608Metric_Pad1.08x0.95mm_HandSolder" (at 77.47 160.02 0)
+      (effects (font (size 1.27 1.27)) hide)
+    )
+    (property "Datasheet" "~" (at 77.47 160.02 0)
+      (effects (font (size 1.27 1.27)) hide)
+    )
