File: PCB_Design/Suspension_telemetry/Power_Stabilizer_5V.kicad_sch (KiCad schematic)
At the start: 6 parts, among them U2 TLV61046ADB

Commit message: adding swnsor mounts
Connections:
- net EN: now reaches U2.4 (EN)
- no-connect marks 1 -> 0
Changed lines of the file:
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@@
   (junction (at 148.59 53.34) (diameter 0) (color 0 0 0 0)
   )
-  (no_connect (at 129.54 67.31))
+  (wire (pts (xy 111.76 67.31) (xy 129.54 67.31))
+    (stroke (width 0) (type default))
+  )
   (wire (pts (xy 144.78 67.31) (xy 144.78 71.12))
     (stroke (width 0) (type default))
@@
     (effects (font (size 1.27 1.27)) (justify left))
   )
+  (hierarchical_label "EN" (shape input) (at 111.76 67.31 180) (fields_autoplaced)
+    (effects (font (size 1.27 1.27)) (justify right))
+  )
   (symbol (lib_id "Device:C_Small") (at 118.11 58.42 180) (unit 1)
