File: PCB_Design/Suspension_telemetry/Suspension_telemetry.kicad_pcb (KiCad board)
At the start: 2 copper layers, 85 parts, among them IC1 MCP73844-840I_MS, J1 USB4500-03-0-A, J10 Conn_01x03_Pin, J11 530480310, J12 530480410, J2 Conn_01x03_Pin, J3 112J-TDAR-R01, J4 Conn_02x04_Top_Bottom, J5 HBHR-B2-10-VG-SMT, J6 Conn_01x08_Socket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

Commit message: PCB: Finished
Parts:
- removed H1, H2, H3, H4: MountingHole_Pad, MountingHole:MountingHole_4.3mm_M4_DIN965_Pad_TopBottom
- J10: footprint Connector_PinHeader_2.54mm:PinHeader_1x03_P2.54mm_Vertical -> Connector_PinHeader_1.27mm:PinHeader_1x03_P1.27mm_Vertical
- moved R24 181.8 mm to (78.0, 95.5), turned to 180 degrees
- moved R23 181.2 mm to (78.0, 98.0)
- moved J10 157.7 mm to (110.5, 89.9), turned to 90 degrees
- moved R22 147.4 mm to (110.7, 113.0), turned to 90 degrees
- moved R21 145.1 mm to (113.0, 113.0), turned to -90 degrees
- moved C25 144.7 mm to (125.5, 96.4), turned to -90 degrees
- moved R16 138.3 mm to (121.4, 96.4), turned to -90 degrees
- moved R15 136.8 mm to (123.4, 96.4), turned to -90 degrees
- moved R17 134.4 mm to (131.6, 96.4), turned to -90 degrees
- moved R13 134.1 mm to (127.5, 96.4), turned to -90 degrees
- moved R18 131.8 mm to (133.6, 96.4), turned to -90 degrees
- moved R14 131.5 mm to (129.5, 96.4), turned to -90 degrees
- moved L3 130.9 mm to (76.6, 107.3), turned to 90 degrees
- moved C26 121.2 mm to (77.3, 103.9)
- moved C27 119.6 mm to (77.3, 101.5)
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Connections:
- J1 pad A6: DATAP_CONN -> DATAP
- J1 pad A7: DATAN_CONN -> DATAN
- J1 pad B6: DATAP_CONN -> DATAP
- J1 pad B7: DATAP_CONN -> DATAN
- J1 pad MH1: unconnected-(J1-PadMH1) -> GND
- J1 pad MH2: unconnected-(J1-PadMH2) -> GND
- J1 pad MH3: unconnected-(J1-PadMH3) -> GND
- J1 pad MH4: unconnected-(J1-PadMH4) -> GND
- J6 pad 1: +3.3V -> GND
- J6 pad 2: GND -> +3.3V
- U1 pad 44: USB_OTG_FS_DM -> USB_OTG_FS_D-
- U1 pad 45: USB_OTG_FS_DP -> USB_OTG_FS_D+
- U5 pad 1: DATAN_CONN -> USB_OTG_FS_D+
- U5 pad 3: DATAP_CONN -> USB_OTG_FS_D-
- U5 pad 4: USB_OTG_FS_DP -> DATAN
- U5 pad 6: USB_OTG_FS_DM -> DATAP
Routing:
- net 5V_USB: track 0.00 -> 187.4 mm, vias 0 -> 2
- net +3.3VA: track 0.00 -> 131.1 mm, vias 0 -> 3
- net I2C1_SDA: track 0.00 -> 89.6 mm, vias 0 -> 1
- net ADC3_IN0: track 0.00 -> 84.7 mm, vias 0 -> 2
- net I2C1_SCL: track 0.00 -> 73.5 mm, vias 0 -> 1
- net +3.3V: track 0.00 -> 73.0 mm, vias 0 -> 9
- net ADC2_IN4: track 0.00 -> 67.3 mm, vias 0 -> 2
- net GND: track 0.00 -> 66.2 mm, vias 0 -> 15
- net +5VA: track 0.00 -> 61.3 mm
- net USART_TX: track 0.00 -> 53.2 mm
- net /Power_Stabilizer_3_3V/V_in_P: track 0.00 -> 50.2 mm, vias 0 -> 4
- net Net-(J8-Pad2): track 0.00 -> 45.1 mm, vias 0 -> 1
- net +5V: track 0.00 -> 43.8 mm, vias 0 -> 2
- net ADC2_IN13: track 0.00 -> 41.9 mm, vias 0 -> 2
- net ADC2_IN1: track 0.00 -> 38.7 mm, vias 0 -> 1
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- added copper zone on B.Cu, net +3.3V
- added copper zone on F.Cu, net GND
Other:
- board outline added: 80 x 48.3 mm

Commit message: Initial:GUI
Parts:
- C10, C11, C8, C9: footprint Capacitor_SMD:C_0805_2012Metric_Pad1.18x1.45mm_HandSolder -> Capacitor_SMD:C_1206_3216Metric_Pad1.33x1.80mm_HandSolder
- moved C25 2.29 mm to (127.8, 96.4)
- moved R13 1.78 mm to (125.7, 96.4)
- moved C9 1.10 mm to (93.6, 116.5)
- moved C10 0.89 mm to (79.0, 114.9)
- moved C8 0.42 mm to (101.3, 111.8)
- moved C11 0.38 mm to (78.0, 119.1)
Routing:
- net +3.3V: track 73.0 -> 69.7 mm
- net /Power_Stabilizer_3_3V/V_in_P: track 50.2 -> 52.0 mm
- net SDIO_CK: track 29.4 -> 27.6 mm
- net Net-(D1-K): track 15.6 -> 14.4 mm
- net SDIO_D3: track 18.7 -> 17.7 mm
