File: PCB_Design/Suspension_telemetry/Suspension_telemetry.kicad_pcb (KiCad board)
At the start: 2 copper layers, 80 x 48.3 mm, 81 parts, among them IC1 MCP73844-840I_MS, J1 USB4500-03-0-A, J10 Conn_01x03_Pin, J11 530480310, J12 530480410, J2 Conn_01x03_Pin, J3 112J-TDAR-R01, J4 Conn_02x04_Top_Bottom, J5 HBHR-B2-10-VG-SMT, J6 Conn_01x08_Socket, J7 530480510, J8 530480310, J9 530480410, Q1 SI4435DY, U1 STM32F446RET6, U2 LMR62421XMF, U3 LM1117MP-3.3, U4 LM1117MP-5.0, U5 USBLC6-2SC6, Y1 Crystal_GND24_Small, Y2 ABS07-32.768KHZ-9-T

Commit message: before pcb v2
Connections:
- J3 pad CD1: GND -> SD_detection
- U1 pad 41: unconnected-(U1-PA8-Pad41) -> SD_detection
Routing:
- net SD_detection: track 0.00 -> 24.3 mm, vias 0 -> 2
- net I2C1_SCL: track 73.5 -> 78.6 mm
- net I2C1_SDA: track 89.6 -> 87.9 mm
Changed lines of the file:
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@@
   (net 75 "ADC2_IN14")
   (net 76 "ADC2_IN13")
-  (net 77 "unconnected-(U1-PA8-Pad41)")
+  (net 77 "SD_detection")
   (net 78 "unconnected-(U1-PA9-Pad42)")
   (net 79 "unconnected-(U1-PA10-Pad43)")
@@
       (net 32 "SDIO_D1") (pinfunction "DAT1") (pintype "passive"))
     (pad "CD1" smd rect (at -6.55 -7.25 180) (size 0.7 1.6) (layers "F.Cu" "F.Paste" "F.Mask")
-      (net 3 "GND") (pinfunction "CARD_DETECTION") (pintype "passive"))
+      (net 77 "SD_detection") (pinfunction "CARD_DETECTION") (pintype "passive"))
     (pad "G1" smd rect (at -7.75 -6.75 180) (size 1.2 1.4) (layers "F.Cu" "F.Paste" "F.Mask")
       (net 3 "GND") (pinfunction "GROUND") (pintype "passive"))
@@
       (net 32 "SDIO_D1") (pinfunction "PC9") (pintype "bidirectional"))
     (pad "41" smd roundrect (at 5.675 -0.25) (size 1.55 0.3) (layers "F.Cu" "F.Paste" "F.Mask") (roundrect_rratio 0.25)
-      (net 77 "unconnected-(U1-PA8-Pad41)") (pinfunction "PA8") (pintype "bidirectional+no_connect"))
+      (net 77 "SD_detection") (pinfunction "PA8") (pintype "bidirectional"))
     (pad "42" smd roundrect (at 5.675 -0.75) (size 1.55 0.3) (layers "F.Cu" "F.Paste" "F.Mask") (roundrect_rratio 0.25)
       (net 78 "unconnected-(U1-PA9-Pad42)") (pinfunction "PA9") (pintype "bidirectional+no_connect"))
@@
   (segment (start 109.728 95.1465) (end 108.756 96.1185) (width 0.3) (layer "F.Cu") (net 55))
   (via (at 110.008 103.0778) (size 0.8) (drill 0.4) (layers "F.Cu" "B.Cu") (net 55))
-  (segment (start 130.048 119.554) (end 130.048 108.458) (width 0.25) (layer "B.Cu") (net 55))
-  (segment (start 114.9092 109.0422) (end 125.222 109.0422) (width 0.25) (layer "B.Cu") (net 55))
+  (segment (start 143.8337 80.6494) (end 143.08 79.8957) (width 0.25) (layer "B.Cu") (net 55))
   (segment (start 143.8337 84.20162) (end 143.8337 80.6494) (width 0.25) (layer "B.Cu") (net 55))
+  (segment (start 114.9092 109.0422) (end 125.222 109.0422) (width 0.25) (layer "B.Cu") (net 55))
+  (segment (start 129.714 108.655695) (end 137.668 100.701695) (width 0.25) (layer "B.Cu") (net 55))
   (segment (start 125.222 109.0422) (end 125.222 118.618) (width 0.25) (layer "B.Cu") (net 55))
-  (segment (start 129.714 119.888) (end 130.048 119.554) (width 0.25) (layer "B.Cu") (net 55))
-  (segment (start 134.874 103.632) (end 134.874 90.3224) (width 0.25) (layer "B.Cu") (net 55))
-  (segment (start 126.492 119.888) (end 129.714 119.888) (width 0.25) (layer "B.Cu") (net 55))
-  (segment (start 140.8007 84.3957) (end 143.63962 84.3957) (width 0.25) (layer "B.Cu") (net 55))
-  (segment (start 143.63962 84.3957) (end 143.8337 84.20162) (width 0.25) (layer "B.Cu") (net 55))
+  (segment (start 137.668 90.36732) (end 143.8337 84.20162) (width 0.25) (layer "B.Cu") (net 55))
   (segment (start 125.222 118.618) (end 126.492 119.888) (width 0.25) (layer "B.Cu") (net 55))
-  (segment (start 134.874 90.3224) (end 140.8007 84.3957) (width 0.25) (layer "B.Cu") (net 55))
-  (segment (start 130.048 108.458) (end 134.874 103.632) (width 0.25) (layer "B.Cu") (net 55))
-  (segment (start 143.8337 80.6494) (end 143.08 79.8957) (width 0.25) (layer "B.Cu") (net 55))
+  (segment (start 137.668 100.701695) (end 137.668 90.36732) (width 0.25) (layer "B.Cu") (net 55))
+  (segment (start 126.492 119.888) (end 129.714 119.888) (width 0.25) (layer "B.Cu") (net 55))
+  (segment (start 129.714 119.888) (end 129.714 108.655695) (width 0.25) (layer "B.Cu") (net 55))
   (segment (start 110.008 103.0778) (end 110.008 104.141) (width 0.25) (layer "B.Cu") (net 55))
   (segment (start 110.008 104.141) (end 114.9092 109.0422) (width 0.25) (layer "B.Cu") (net 55))
@@
   (via (at 110.5763 96.6717) (size 0.8) (drill 0.4) (layers "F.Cu" "B.Cu") (net 56))
   (segment (start 111.5888 96.6717) (end 110.5763 96.6717) (width 0.25) (layer "B.Cu") (net 56))
-  (segment (start 129.032 107.442) (end 133.2648 103.2092) (width 0.25) (layer "B.Cu") (net 56))
-  (segment (start 133.2648 103.2092) (end 133.2648 90.9609) (width 0.25) (layer "B.Cu") (net 56))
-  (segment (start 133.2648 92.456) (end 115.8045 92.456) (width 0.25) (layer "B.Cu") (net 56))
+  (segment (start 127.762 118.618) (end 127.762 108.712) (width 0.25) (layer "B.Cu") (net 56))
+  (segment (start 122.564305 92.456) (end 127.192605 87.8277) (width 0.25) (layer "B.Cu") (net 56))
+  (segment (start 115.8045 92.456) (end 122.564305 92.456) (width 0.25) (layer "B.Cu") (net 56))
+  (segment (start 136.398 100.076) (end 136.398 87.8277) (width 0.25) (layer "B.Cu") (net 56))
   (segment (start 115.8045 92.456) (end 111.5888 96.6717) (width 0.25) (layer "B.Cu") (net 56))
-  (segment (start 133.2648 90.9609) (end 143.08 81.1457) (width 0.25) (layer "B.Cu") (net 56))
-  (segment (start 129.032 116.078) (end 129.032 107.442) (width 0.25) (layer "B.Cu") (net 56))
-  (segment (start 127.762 118.618) (end 127.762 117.348) (width 0.25) (layer "B.Cu") (net 56))
-  (segment (start 127.762 117.348) (end 129.032 116.078) (width 0.25) (layer "B.Cu") (net 56))
+  (segment (start 127.762 108.712) (end 136.398 100.076) (width 0.25) (layer "B.Cu") (net 56))
+  (segment (start 136.398 87.8277) (end 143.08 81.1457) (width 0.25) (layer "B.Cu") (net 56))
+  (segment (start 127.192605 87.8277) (end 136.398 87.8277) (width 0.25) (layer "B.Cu") (net 56))
   (segment (start 139.7705 82.3957) (end 138.9911 83.1751) (width 0.25) (layer "F.Cu") (net 57))
   (segment (start 143.08 82.3957) (end 139.7705 82.3957) (width 0.25) (layer "F.Cu") (net 57))
@@
   (segment (start 92.075 104.2162) (end 92.0792 104.212) (width 0.25) (layer "B.Cu") (net 76))
   (segment (start 92.0792 104.212) (end 107.3097 104.212) (width 0.25) (layer "B.Cu") (net 76))
+  (segment (start 119.38 103.124) (end 118.614 103.89) (width 0.25) (layer "F.Cu") (net 77))
+  (segment (start 118.614 103.89) (end 117.181 103.89) (width 0.25) (layer "F.Cu") (net 77))
+  (segment (start 133.804 89.608) (end 133.604 89.408) (width 0.25) (layer "F.Cu") (net 77))
+  (segment (start 133.804 91.161) (end 133.804 89.608) (width 0.25) (layer "F.Cu") (net 77))
+  (via (at 119.38 103.124) (size 0.8) (drill 0.4) (layers "F.Cu" "B.Cu") (net 77))
+  (via (at 133.604 89.408) (size 0.8) (drill 0.4) (layers "F.Cu" "B.Cu") (net 77))
+  (segment (start 133.096 89.408) (end 119.38 103.124) (width 0.25) (layer "B.Cu") (net 77))
+  (segment (start 133.604 89.408) (end 133.096 89.408) (width 0.25) (layer "B.Cu") (net 77))
   (segment (start 131.196 101.534) (end 131.1965 101.534) (width 0.25) (layer "F.Cu") (net 81))
   (segment (start 131.196 101.534) (end 129.937 101.534) (width 0.25) (layer "F.Cu") (net 81))

Commit message: pcv v2 finished
Parts:
- removed C11: 10uF, Capacitor_SMD:C_1206_3216Metric_Pad1.33x1.80mm_HandSolder
- removed C21: 0.1u, Capacitor_SMD:C_0603_1608Metric
- removed D1, D3: B240, Diode_SMD:D_SMB
- removed J10: Conn_01x03_Pin, Connector_PinHeader_1.27mm:PinHeader_1x03_P1.27mm_Vertical
- removed J11, J8: 530480310, molex_conn:530480310
- removed J12, J9: 530480410, molex_conn:530480410
- removed J6: Conn_01x08_Socket, Connector_PinSocket_2.54mm:PinSocket_1x08_P2.54mm_Vertical
- removed locked (x2): locked, BAT_BK-18650-PC2:BAT_BK-18650-PC2
- added BT2: BK-18650-PC2, BAT_BK-18650-PC2:BAT_BK-18650-PC2, F.Cu at (106.8, 109.9)
- added N1: Housing, Symbol:CE-Logo_8.5x6mm_SilkScreen, B.Cu at (107.5, 58.7)
- added N2: Housing, Symbol:CE-Logo_8.5x6mm_SilkScreen, B.Cu at (61.0, 84.3)
- added N3: Housing, Symbol:CE-Logo_8.5x6mm_SilkScreen, B.Cu at (140.0, 66.5)
- added R25: 4,7k, Resistor_SMD:R_0603_1608Metric_Pad0.98x0.95mm_HandSolder, B.Cu at (93.7, 99.4)
- added R27: 1k, Resistor_SMD:R_0603_1608Metric_Pad0.98x0.95mm_HandSolder, B.Cu at (122.6, 99.5)
- added R29: 1k, Resistor_SMD:R_0603_1608Metric_Pad0.98x0.95mm_HandSolder, B.Cu at (129.0, 99.5)
- added U6: AT24CS254-SSHM, Package_SO:SOIC-8_3.9x4.9mm_P1.27mm, B.Cu at (76.6, 84.8)
- C1, C2, C6: value 10uF -> 1uF; moved to B.Cu
- C10: value 10uF -> 100n; footprint Capacitor_SMD:C_1206_3216Metric_Pad1.33x1.80mm_HandSolder -> Capacitor_SMD:C_0603_1608Metric_Pad1.08x0.95mm_HandSolder; moved to B.Cu
- C12, C13, C14, C15, C16, C17, C18, C19, C20, C22, C23, C24, C26, C27, C8, C9, D2, L2, L3, R11, R12, R19, R20, R21, R22, R3, R8, R9, U1, U3, U5, Y1, Y2: moved to B.Cu
- C3: value 1n -> 1uF; moved to B.Cu
- C4, C5: value 10uF -> 100n; moved to B.Cu
- C7: value 0.1uF -> 100n; moved to B.Cu
- IC1: value MCP73844-840I_MS -> MCP73114-0NSI_MF; footprint SOP65P490X110-8N:SOP65P490X110-8N -> MCP73114:SON50P300X300X100-11N-D; moved to B.Cu
- J1: value USB4500-03-0-A -> USB3505-30-A_REVA4; footprint USB4500030A:USB4500030A -> GCT_USB3505-30-A_REVA4:GCT_USB3505-30-A_REVA4
- J2: value Conn_01x03_Pin -> 125SH-A-04-TS; footprint Connector_PinHeader_1.27mm:PinHeader_1x03_P1.27mm_Vertical -> molex_conn:125SHA04TS
- J4: value Conn_02x04_Top_Bottom -> 530481010; footprint Connector_PinSocket_2.54mm:PinSocket_2x04_P2.54mm_Vertical -> MOLEX_10_PIN:530481010
- J5: value HBHR-B2-10-VG-SMT -> 280384-1; footprint HBHRB210VGSMT:HBHRB210VGSMT -> BUTTON_CONN:2803841
- J7: value 530480510 -> Conn_02x03_Top_Bottom; footprint molex_conn:530480510 -> Connector_PinHeader_2.54mm:PinHeader_2x03_P2.54mm_Vertical
- L1: value DR73-6R8-R -> LQH3NPZ100MJRL; footprint INDM7676X355N:INDM7676X355N -> LQH3NPN100MJRL:LQH3NPN100MJRL; moved to B.Cu
- Q1: value SI4435DY -> AOSP32368; footprint SOIC127P600X175-8N:SOIC127P600X175-8N -> footprints:SO8SOP-8L_AOS; moved to B.Cu
- R1: value 10k -> 1.1k; moved to B.Cu
- R10: value 22 -> 10k; moved to B.Cu
- R2: value 1M -> 360k; moved to B.Cu
- R23: value 6,8k -> 4,7k; moved to B.Cu
- R24: value 4,7k -> 6,8k; moved to B.Cu
- R4: value 100k -> 1k; moved to B.Cu
- R5: value 100m -> 10k; moved to B.Cu
- R6, R7: value 5,1k -> 100k; moved to B.Cu
- S1: value 1825965-1 -> OS102011MA1QN1; footprint 18259651-switch:18259651 -> MikroP_90:OS102011MA1QN1
- U2: value LMR62421XMF -> TLV61046ADB; footprint Package_TO_SOT_SMD:SOT-23-5 -> Package_TO_SOT_SMD:SOT-23-6; moved to B.Cu
- U4: value LM1117MP-5.0 -> ADXL343; footprint Package_TO_SOT_SMD:SOT-223-3_TabPin2 -> Package_LGA:LGA-14_3x5mm_P0.8mm_LayoutBorder1x6y; moved to B.Cu
- moved C6 66.2 mm to (142.3, 103.1)
- moved R19 59.6 mm to (78.9, 91.8)
- moved IC1 57.3 mm to (138.1, 103.5)
- moved R5 56.4 mm to (142.1, 117.5), turned to 180 degrees
- moved C1 54.9 mm to (138.1, 100.3), turned to 0 degrees
- moved L1 51.9 mm to (128.3, 108.2)
- moved R4 50.6 mm to (132.6, 104.6), turned to 180 degrees
- moved R1 50.4 mm to (134.3, 101.3), turned to 90 degrees
- moved R2 50.0 mm to (122.9, 117.6)
- moved U2 49.2 mm to (128.3, 112.3)
- moved R3 47.0 mm to (126.6, 118.5)
- moved J4 46.0 mm to (91.9, 96.4), turned to 0 degrees
- moved D2 45.9 mm to (131.7, 101.3)
- moved C7 44.8 mm to (126.7, 99.5), turned to -90 degrees
- moved Q1 44.3 mm to (135.5, 116.2), turned to 180 degrees
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Connections:
- C10 pad 1: /Power_Stabilizer_3_3V/V_in_P -> PWR_SWITCH_OUT
- C2 pad 1: Net-(D1-K) -> GND
- C2 pad 2: GND -> /Power_Stabilizer_3_3V/V_in_P
- C3 pad 1: Net-(D1-K) -> GND
- C3 pad 2: Net-(U2-FB) -> +5V
- C4 pad 1: Net-(D1-K) -> RIGHT_BUTTON
- C5 pad 1: Net-(D2-A) -> NRST
- C7 pad 1: Net-(IC1-TIMER) -> LEFT_BUTTON
- D2 pad 2: Net-(D2-A) -> 5V_USB
- IC1 pad 1: Net-(IC1-SENSE) -> 5V_USB
- IC1 pad 2: Net-(D2-A) -> 5V_USB
- IC1 pad 3: Net-(D2-K) -> /Power_Stabilizer_3_3V/V_in_P
- IC1 pad 4: Net-(IC1-EN) -> /Power_Stabilizer_3_3V/V_in_P
- IC1 pad 5: Net-(IC1-TIMER) -> unconnected-(IC1-NC_1-Pad5)
- IC1 pad 6: GND -> unconnected-(IC1-NC_2-Pad6)
- IC1 pad 7: /Power_Stabilizer_3_3V/V_in_P -> Net-(IC1-STAT)
- IC1 pad 8: Net-(IC1-DRV) -> GND
- J2 pad 1: +3.3V -> I2C1_SDA
- J2 pad 2: Net-(J2-Pin_2) -> I2C1_SCL
- J4 pad 1: GND -> PRESSURE_FRONT_OUT
- J4 pad 2: USART_RX -> PRESSURE_REAR_OUT
- J4 pad 3: unconnected-(J4-Pin_3-Pad3) -> GND
- J4 pad 4: ESP8266_CH_PD -> +3.3VA
- J4 pad 5: unconnected-(J4-Pin_5-Pad5) -> TRAVEL_SENOR_REAR
- J4 pad 6: unconnected-(J4-Pin_6-Pad6) -> TRAVEL_SENSOR_FRONT
- J4 pad 7: USART_TX -> BRAKE_SENSOR_LEFT
- J4 pad 8: +3.3V -> BRAKE_SENSOR_RIGHT
- J5 pad 1: +3.3V -> GND
- J5 pad 2: Net-(J5-SWDIO) -> +3.3V
- J5 pad 3: GND -> LB_PRE_DEB
- J5 pad 4: SWDCLK -> PWR_SWITCH_IN
- J5 pad 5: GND -> RB_PRE_DEB
- J5 pad 6: SWO -> PWR_SWITCH_OUT
- J5 pad 7: unconnected-(J5-KEY-Pad7) -> NRST
- J5 pad 8: unconnected-(J5-NC/EXTb-Pad8) -> GND
- J7 pad 1: GND -> NRST
- J7 pad 2: Net-(J10-Pin_2) -> +3.3V
- J7 pad 3: I2C1_SCL -> GND
- J7 pad 4: I2C1_SDA -> SWO
- J7 pad 5: Net-(J7-Pad5) -> SWDIO
- L1 pad 1: 5V_USB -> /Power_Stabilizer_3_3V/V_in_P
- Q1 pad 1: Net-(IC1-SENSE) -> GND
- Q1 pad 2: Net-(IC1-SENSE) -> GND
- Q1 pad 3: Net-(IC1-SENSE) -> GND
- Q1 pad 4: Net-(IC1-DRV) -> Net-(Q1-Pad4)
- Q1 pad 5: /Power_Stabilizer_3_3V/V_in_P -> PWR_SWITCH_IN
- Q1 pad 6: /Power_Stabilizer_3_3V/V_in_P -> PWR_SWITCH_IN
- Q1 pad 7: /Power_Stabilizer_3_3V/V_in_P -> PWR_SWITCH_IN
- Q1 pad 8: /Power_Stabilizer_3_3V/V_in_P -> PWR_SWITCH_IN
- R1 pad 1: Net-(U2-FB) -> Net-(IC1-PROG)
- R10 pad 1: Net-(J5-SWDIO) -> GND
- R10 pad 2: SWDIO -> Net-(U4-SDO/ADDR)
- R19 pad 1: Net-(J7-Pad5) -> +3.3V
- R19 pad 2: ADC3_IN0 -> Net-(U4-~{CS})
- R2 pad 1: 5V_USB -> +5V
- R2 pad 2: Net-(U2-EN) -> Net-(U2-FB)
- R20 pad 1: ADC3_IN0 -> CHARGE_DETECTION
- R21 pad 1: ADC2_IN14 -> PRESSURE_SENSOR_REAR
- R22 pad 1: Net-(J8-Pad2) -> PRESSURE_REAR_OUT
- R22 pad 2: ADC2_IN14 -> PRESSURE_SENSOR_REAR
- R23 pad 1: ADC2_IN13 -> 5V_USB
- R23 pad 2: GND -> CHARGE_DETECTION
- R24 pad 1: Net-(J11-Pad2) -> PRESSURE_SENSOR_FRONT
- R24 pad 2: ADC2_IN13 -> GND
- R3 pad 1: Net-(D1-K) -> GND
- R4 pad 1: Net-(IC1-EN) -> Net-(IC1-STAT)
- R4 pad 2: Net-(D2-A) -> Net-(D2-K)
- R5 pad 1: Net-(D2-A) -> /Power_Stabilizer_3_3V/V_in_P
- R5 pad 2: Net-(IC1-SENSE) -> Net-(Q1-Pad4)
- R6 pad 1: GND -> BATTERY_LEVEL
- R6 pad 2: CC2 -> /Power_Stabilizer_3_3V/V_in_P
- R7 pad 2: CC1 -> BATTERY_LEVEL
- R9 pad 1: Net-(J2-Pin_2) -> Net-(R9-Pad1)
- S1 pad 1: NRST -> GND
- S1 pad 2: GND -> Net-(R9-Pad1)
- U1 pad 10: unconnected-(U1-PC2-Pad10) -> TRAVEL_SENSOR_FRONT
- U1 pad 11: ADC2_IN13 -> TRAVEL_SENOR_REAR
- U1 pad 14: ADC3_IN0 -> unconnected-(U1-PA0-Pad14)
- U1 pad 15: ADC2_IN1 -> PRESSURE_SENSOR_FRONT
- U1 pad 16: USART_TX -> PRESSURE_SENSOR_REAR
- U1 pad 17: USART_RX -> unconnected-(U1-PA3-Pad17)
- U1 pad 20: ADC2_IN4 -> BATTERY_LEVEL
- U1 pad 21: PA5 -> unconnected-(U1-PA5-Pad21)
- U1 pad 24: ADC2_IN14 -> unconnected-(U1-PC4-Pad24)
- U1 pad 26: ESP8266_CH_PD -> unconnected-(U1-PB0-Pad26)
- U1 pad 38: unconnected-(U1-PC7-Pad38) -> ACCELEROMETER_INT0
- U1 pad 50: unconnected-(U1-PA15-Pad50) -> CHARGE_DETECTION
- U1 pad 58: unconnected-(U1-PB6-Pad58) -> RIGHT_BUTTON
- U1 pad 59: unconnected-(U1-PB7-Pad59) -> LEFT_BUTTON
- U1 pad 8: unconnected-(U1-PC0-Pad8) -> BRAKE_SENSOR_RIGHT
- U1 pad 9: unconnected-(U1-PC1-Pad9) -> BRAKE_SENSOR_LEFT
- U2 pad 4: Net-(U2-EN) -> unconnected-(U2-EN-Pad4)
- U2 pad 5: 5V_USB -> +5V
- U4 pad 1: GND -> +3.3V
- U4 pad 2: +5V -> GND
- U4 pad 3: /Power_Stabilizer_3_3V/V_in_P -> unconnected-(U4-RES-Pad3)
Routing:
- net PWR_SWITCH_OUT: track 0.00 -> 141.2 mm
- net +3.3VA: track 131.0 -> 21.8 mm, vias 3 -> 0
- net 5V_USB: track 187.4 -> 78.6 mm
- net GND: track 65.8 -> 157.9 mm, vias 15 -> 32
- net ADC3_IN0: track 84.7 -> 0.00 mm, vias 2 -> 0
- net SDIO_D3: track 17.7 -> 89.9 mm, vias 2 -> 1
- net ADC2_IN4: track 67.3 -> 0.00 mm, vias 2 -> 0
- net USART_TX: track 53.2 -> 0.00 mm
- net PWR_SWITCH_IN: track 0.00 -> 51.8 mm
- net +5VA: track 61.2 -> 11.3 mm
- net ACCELEROMETER_INT0: track 0.00 -> 48.2 mm, vias 0 -> 2
- net Net-(J8-Pad2): track 45.1 -> 0.00 mm, vias 1 -> 0
- net ADC2_IN13: track 41.9 -> 0.00 mm, vias 2 -> 0
- net LEFT_BUTTON: track 0.00 -> 38.8 mm, vias 0 -> 2
- net ADC2_IN1: track 38.7 -> 0.00 mm, vias 1 -> 0
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- added copper zone on F.Cu, net +3.3V
- added copper zone on B.Cu, net GND
- removed copper zone on B.Cu, net +3.3V
- removed copper zone on F.Cu, net GND
Other:
- board size 80 x 48.3 mm -> 75.9 x 50.1 mm
- board text added: "3.3V"
- board text added: "5V"
- board text added: "BL"
- board text added: "BOOT_OFF"
- board text added: "BOOT_ON"
- board text added: "BR"
- board text added: "DIO"
- board text added: "GND"
- board text added: "LB"
- board text added: "NRST"
- board text added: "PF"
- board text added: "POUT"
- board text added: "PR"
- board text added: "PWIN"
- board text added: "RB"
- board text added: "SCLK"
- board text added: "SWO"
- board text added: "TF"
- board text added: "TR"
