File: PCB_Design/Suspension_telemetry/Power_Stabilizer_3_3V.kicad_sch (KiCad schematic)
At the start: 3 parts, among them U3 LM1117MP-3.3

Commit message: Initial:GUI
Parts:
- C8, C9: footprint Capacitor_SMD:C_0805_2012Metric_Pad1.18x1.45mm_HandSolder -> Capacitor_SMD:C_1206_3216Metric_Pad1.33x1.80mm_HandSolder
Changed lines of the file:
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@@
       (effects (font (size 1.27 1.27)) (justify left))
     )
-    (property "Footprint" "Capacitor_SMD:C_0805_2012Metric_Pad1.18x1.45mm_HandSolder" (at 154.94 63.5 0)
+    (property "Footprint" "Capacitor_SMD:C_1206_3216Metric_Pad1.33x1.80mm_HandSolder" (at 154.94 63.5 0)
       (effects (font (size 1.27 1.27)) hide)
     )
@@
       (effects (font (size 1.27 1.27)) (justify left))
     )
-    (property "Footprint" "Capacitor_SMD:C_0805_2012Metric_Pad1.18x1.45mm_HandSolder" (at 110.49 63.5 0)
+    (property "Footprint" "Capacitor_SMD:C_1206_3216Metric_Pad1.33x1.80mm_HandSolder" (at 110.49 63.5 0)
       (effects (font (size 1.27 1.27)) hide)
     )

Commit message: pcv v2 finished
Connections:
- net V_Out_M renamed GND
Changed lines of the file:
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@@
   (junction (at 110.49 58.42) (diameter 0) (color 0 0 0 0)
-  )
-  (junction (at 154.94 71.12) (diameter 0) (color 0 0 0 0)
-  )
-  (junction (at 110.49 71.12) (diameter 0) (color 0 0 0 0)
   )
   (junction (at 132.08 71.12) (diameter 0) (color 0 0 0 0)
@@
   )
   (wire (pts (xy 154.94 71.12) (xy 132.08 71.12))
+    (stroke (width 0) (type default))
+  )
+  (wire (pts (xy 132.08 71.12) (xy 132.08 74.93))
     (stroke (width 0) (type default))
   )
@@
     (stroke (width 0) (type default))
   )
-  (wire (pts (xy 154.94 71.12) (xy 161.29 71.12))
-    (stroke (width 0) (type default))
-  )
   (wire (pts (xy 132.08 66.04) (xy 132.08 71.12))
-    (stroke (width 0) (type default))
-  )
-  (wire (pts (xy 101.6 71.12) (xy 110.49 71.12))
     (stroke (width 0) (type default))
   )
@@
   (hierarchical_label "V_Out_P" (shape output) (at 161.29 58.42 0) (fields_autoplaced)
     (effects (font (size 1.27 1.27)) (justify left))
-  )
-  (hierarchical_label "V_Out_M" (shape output) (at 161.29 71.12 0) (fields_autoplaced)
-    (effects (font (size 1.27 1.27)) (justify left))
-  )
-  (hierarchical_label "V_in_M" (shape input) (at 101.6 71.12 180) (fields_autoplaced)
-    (effects (font (size 1.27 1.27)) (justify right))
   )
   (symbol (lib_id "Regulator_Linear:LM1117MP-3.3") (at 132.08 58.42 0) (unit 1)
@@
         )
       )
+    )
+  )
+  (symbol (lib_id "power:GND") (at 132.08 74.93 0) (unit 1)
+    (in_bom yes) (on_board yes) (dnp no) (fields_autoplaced)
+    (property "Reference" "#PWR04" (at 132.08 81.28 0)
+      (effects (font (size 1.27 1.27)) hide)
+    )
+    (property "Value" "GND" (at 132.08 80.01 0)
+      (effects (font (size 1.27 1.27)))
+    )
+    (property "Footprint" "" (at 132.08 74.93 0)
+      (effects (font (size 1.27 1.27)) hide)
+    )
+    (property "Datasheet" "" (at 132.08 74.93 0)
+      (effects (font (size 1.27 1.27)) hide)
+    )
+    (pin "1")
+    (instances
+      (project "Suspension_telemetry"
+        (path "/5c831aae-4894-4c31-a571-d996f699966b/662b9913-71f4-469d-b95c-3a768392d596"
+          (reference "#PWR04") (unit 1)
+        )
+        (path "/5c831aae-4894-4c31-a571-d996f699966b/cd1ff58d-48eb-463d-8546-c9aeb7c83a06"
+          (reference "#PWR018") (unit 1)
+        )
+        (path "/5c831aae-4894-4c31-a571-d996f699966b/827d91e7-d2fd-441d-a7c6-e88b25daf035"
+          (reference "#PWR07") (unit 1)
+        )
+      )
