File: PCB_Design/Suspension_telemetry/USB_C.kicad_sch (KiCad schematic)
At the start: 3 parts, among them J1 USB4500-03-0-A

Commit message: PCB: Finished
Connections:
- net DN2: now also J1.B7 (DN2)
- net DP2: no longer J1.B7 (DN2)
- net GND: now also J1.MH1, J1.MH2, J1.MH3, J1.MH4
- no-connect marks 6 -> 2
Changed lines of the file:
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@@
   (junction (at 101.6 69.85) (diameter 0) (color 0 0 0 0)
   )
+  (junction (at 161.29 80.01) (diameter 0) (color 0 0 0 0)
+  )
+  (junction (at 161.29 85.09) (diameter 0) (color 0 0 0 0)
+  )
   (junction (at 128.27 96.52) (diameter 0) (color 0 0 0 0)
   )
   (junction (at 114.3 74.93) (diameter 0) (color 0 0 0 0)
   )
+  (junction (at 161.29 82.55) (diameter 0) (color 0 0 0 0)
+  )
   (junction (at 69.85 78.74) (diameter 0) (color 0 0 0 0)
   )
   (junction (at 128.27 85.09) (diameter 0) (color 0 0 0 0)
   )
-  (no_connect (at 160.02 77.47))
+  (junction (at 143.51 96.52) (diameter 0) (color 0 0 0 0)
+  )
   (no_connect (at 129.54 80.01))
-  (no_connect (at 160.02 82.55))
-  (no_connect (at 160.02 80.01))
   (no_connect (at 160.02 74.93))
-  (no_connect (at 160.02 85.09))
   (wire (pts (xy 101.6 82.55) (xy 101.6 69.85))
     (stroke (width 0) (type default))
@@
     (stroke (width 0) (type default))
   )
+  (wire (pts (xy 143.51 96.52) (xy 161.29 96.52))
+    (stroke (width 0) (type default))
+  )
   (wire (pts (xy 67.31 78.74) (xy 69.85 78.74))
     (stroke (width 0) (type default))
@@
     (stroke (width 0) (type default))
   )
+  (wire (pts (xy 160.02 82.55) (xy 161.29 82.55))
+    (stroke (width 0) (type default))
+  )
+  (wire (pts (xy 161.29 96.52) (xy 161.29 85.09))
+    (stroke (width 0) (type default))
+  )
+  (wire (pts (xy 161.29 77.47) (xy 161.29 80.01))
+    (stroke (width 0) (type default))
+  )
   (wire (pts (xy 113.03 74.93) (xy 114.3 74.93))
     (stroke (width 0) (type default))
@@
     (stroke (width 0) (type default))
   )
+  (wire (pts (xy 128.27 96.52) (xy 113.03 96.52))
+    (stroke (width 0) (type default))
+  )
+  (wire (pts (xy 125.73 72.39) (xy 129.54 72.39))
+    (stroke (width 0) (type default))
+  )
+  (wire (pts (xy 72.39 78.74) (xy 69.85 78.74))
+    (stroke (width 0) (type default))
+  )
+  (wire (pts (xy 143.51 96.52) (xy 143.51 100.33))
+    (stroke (width 0) (type default))
+  )
+  (wire (pts (xy 113.03 77.47) (xy 116.84 77.47))
+    (stroke (width 0) (type default))
+  )
+  (wire (pts (xy 128.27 96.52) (xy 128.27 99.06))
+    (stroke (width 0) (type default))
+  )
+  (wire (pts (xy 160.02 85.09) (xy 161.29 85.09))
+    (stroke (width 0) (type default))
+  )
+  (wire (pts (xy 129.54 82.55) (xy 101.6 82.55))
+    (stroke (width 0) (type default))
+  )
+  (wire (pts (xy 128.27 67.31) (xy 128.27 85.09))
+    (stroke (width 0) (type default))
+  )
+  (wire (pts (xy 161.29 82.55) (xy 161.29 80.01))
+    (stroke (width 0) (type default))
+  )
+  (wire (pts (xy 114.3 74.93) (xy 129.54 74.93))
+    (stroke (width 0) (type default))
+  )
+  (wire (pts (xy 160.02 67.31) (xy 163.83 67.31))
+    (stroke (width 0) (type default))
+  )
+  (wire (pts (xy 160.02 77.47) (xy 161.29 77.47))
+    (stroke (width 0) (type default))
+  )
+  (wire (pts (xy 114.3 74.93) (xy 114.3 90.17))
+    (stroke (width 0) (type default))
+  )
+  (wire (pts (xy 101.6 69.85) (xy 129.54 69.85))
+    (stroke (width 0) (type default))
+  )
+  (wire (pts (xy 161.29 85.09) (xy 161.29 82.55))
+    (stroke (width 0) (type default))
+  )
+  (wire (pts (xy 67.31 69.85) (xy 67.31 73.66))
+    (stroke (width 0) (type default))
+  )
+  (wire (pts (xy 116.84 77.47) (xy 129.54 77.47))
+    (stroke (width 0) (type default))
+  )
+  (wire (pts (xy 97.79 69.85) (xy 101.6 69.85))
+    (stroke (width 0) (type default))
+  )
+  (wire (pts (xy 160.02 72.39) (xy 163.83 72.39))
+    (stroke (width 0) (type default))
+  )
+  (wire (pts (xy 161.29 80.01) (xy 160.02 80.01))
+    (stroke (width 0) (type default))
+  )
+  (wire (pts (xy 97.79 99.06) (xy 128.27 99.06))
+    (stroke (width 0) (type default))
+  )
   (wire (pts (xy 128.27 96.52) (xy 143.51 96.52))
     (stroke (width 0) (type default))
   )
-  (wire (pts (xy 125.73 72.39) (xy 129.54 72.39))
-    (stroke (width 0) (type default))
-  )
-  (wire (pts (xy 72.39 78.74) (xy 69.85 78.74))
-    (stroke (width 0) (type default))
-  )
-  (wire (pts (xy 143.51 96.52) (xy 143.51 100.33))
-    (stroke (width 0) (type default))
-  )
-  (wire (pts (xy 113.03 77.47) (xy 116.84 77.47))
-    (stroke (width 0) (type default))
-  )
-  (wire (pts (xy 128.27 96.52) (xy 128.27 99.06))
-    (stroke (width 0) (type default))
-  )
-  (wire (pts (xy 129.54 82.55) (xy 101.6 82.55))
-    (stroke (width 0) (type default))
-  )
-  (wire (pts (xy 128.27 67.31) (xy 128.27 85.09))
-    (stroke (width 0) (type default))
-  )
-  (wire (pts (xy 114.3 74.93) (xy 129.54 74.93))
-    (stroke (width 0) (type default))
-  )
-  (wire (pts (xy 160.02 67.31) (xy 163.83 67.31))
-    (stroke (width 0) (type default))
-  )
-  (wire (pts (xy 114.3 74.93) (xy 114.3 90.17))
-    (stroke (width 0) (type default))
-  )
-  (wire (pts (xy 101.6 69.85) (xy 129.54 69.85))
-    (stroke (width 0) (type default))
-  )
-  (wire (pts (xy 67.31 69.85) (xy 67.31 73.66))
-    (stroke (width 0) (type default))
-  )
-  (wire (pts (xy 116.84 77.47) (xy 129.54 77.47))
-    (stroke (width 0) (type default))
-  )
-  (wire (pts (xy 97.79 69.85) (xy 101.6 69.85))
-    (stroke (width 0) (type default))
-  )
-  (wire (pts (xy 160.02 72.39) (xy 163.83 72.39))
-    (stroke (width 0) (type default))
-  )
-  (wire (pts (xy 97.79 99.06) (xy 128.27 99.06))
-    (stroke (width 0) (type default))
-  )
   (wire (pts (xy 129.54 67.31) (xy 128.27 67.31))
     (stroke (width 0) (type default))
@@
     (stroke (width 0) (type default))
   )
-  (global_label "DP2" (shape bidirectional) (at 163.83 72.39 0) (fields_autoplaced)
-    (effects (font (size 1.27 1.27)) (justify left))
-    (property "Intersheetrefs" "${INTERSHEET_REFS}" (at 171.676 72.39 0)
+  (global_label "DN2" (shape bidirectional) (at 163.83 72.39 0) (fields_autoplaced)
+    (effects (font (size 1.27 1.27)) (justify left))
+    (property "Intersheetrefs" "${INTERSHEET_REFS}" (at 171.7365 72.39 0)
       (effects (font (size 1.27 1.27)) (justify left) hide)
     )
@@
     )
   )
-  (symbol (lib_id "power:GND") (at 143.51 100.33 0) (unit 1)
-    (in_bom yes) (on_board yes) (dnp no) (fields_autoplaced)
+  (symbol (lib_id "power:GND") (at 143.51 100.33 0) (mirror y) (unit 1)
+    (in_bom yes) (on_board yes) (dnp no)
     (property "Reference" "#PWR06" (at 143.51 106.68 0)
       (effects (font (size 1.27 1.27)) hide)

Commit message: pcv v2 finished
Parts:
- removed J1: USB4500-03-0-A, USB4500030A:USB4500030A, symbol USB4500-03-0-A:USB4500-03-0-A
- removed R6, R7: 5,1k, Resistor_SMD:R_0603_1608Metric_Pad0.98x0.95mm_HandSolder, symbol Device:R_Small
- added J1: USB3505-30-A_REVA4, GCT_USB3505-30-A_REVA4:GCT_USB3505-30-A_REVA4, symbol USB_micro_water:USB3505-30-A_REVA4
Connections:
- net GND: now also J1.5 (GND), J1.S1 (SHIELD), J1.S2 (SHIELD), J1.S3 (SHIELD), J1.S4 (SHIELD)
- new net 5V: J1.1 (VCC)
- new net DATAN: J1.2 (D-)
- new net DATAP: J1.3 (D+)
- no-connect marks 2 -> 1
